Commit message: feat(inspectra_description): Gazebo + MoveIt fully integrated (Feature 7b-ii COMPLETE)
Chain of fixes required to get here, in order:
- Fixed Command()/xacro pipe bug via standalone generate_panda_urdf.sh
- Reapplied franka_description fer/inertials.yaml link4 workaround
  (known upstream bug, had silently reverted between sessions)
- Fixed <robot name> mismatch: our URDF said 'inspectra_panda', SRDF
  expected 'panda' -- move_group was crashing outright on this
- Switched to MoveItConfigsBuilder pattern (matching demo.launch.py)
  instead of hand-rolled yaml loading, fixing ompl.* namespace crash
- Fixed franka_description fer/joint_limits.yaml joint4 upper bound:
  original -0.0698 caused FP-precision 'outside bounds' rejection
- Root-caused and fixed missing initial joint positions in our
  <ros2_control> block -- without them, joint4 defaulted to sit
  exactly on its limit boundary; added correct initial_value params
  matching moveit_resources' initial_positions.yaml
- Enabled acceleration limits in inspectra_moveit_config's
  joint_limits.yaml (were has_acceleration_limits: false everywhere,
  blocking AddTimeOptimalParameterization)
- Bridged Gazebo's /clock into ROS2 via ros_gz_bridge parameter_bridge
  (use_sim_time nodes were otherwise stalling silently)
- Diagnosed 'start point deviates from current robot state' as a
  self-inflicted state desync from manual controller testing between
  Plan and Execute -- not a real bug, resolved by a clean Plan->Execute
  cycle

VERIFIED END-TO-END: Plan succeeds, Execute succeeds, real physics-based
motion confirmed in both RViz and Gazebo simultaneously, driven through
the actual panda_arm_controller FollowJointTrajectory action -- not
RViz's fake controller.

File: ros2_ws/src/inspectra_description/urdf/inspectra_panda.urdf.xacro (robot description, xacro)
@@ -1,9 +1,9 @@
 <?xml version="1.0"?>
-<robot xmlns:xacro="http://www.ros.org/wiki/xacro" name="inspectra_panda">
+<robot xmlns:xacro="http://www.ros.org/wiki/xacro" name="panda">
   <!-- franka_description (current layout): Panda is now called "fer"
        (Franka Emika Research robot). Joints get prefixed "fer_" by
-       default (fer_joint1..7, fer_link0..8). This differs from
-       moveit_resources_panda_moveit_config's "panda_*" naming used
-       elsewhere in this project — reconciling that is Feature 7b. -->
+       default (fer_joint1..7, fer_link0..8), later renamed to "panda_*"
+       via generate_panda_urdf.sh so names match moveit_resources_panda_
+       moveit_config's SRDF/kinematics/joint_limits. -->
   <xacro:include filename="$(find franka_description)/robots/common/franka_robot.xacro"/>
   <xacro:franka_robot
@@ -16,24 +16,31 @@
   />
   <!-- ros2_control interface: exposes each joint's position command/state
-       so gz_ros2_control's plugin (below) can drive them in simulation. -->
+       so gz_ros2_control's plugin (below) can drive them in simulation.
+       initial_value set explicitly per joint (matching moveit_resources_
+       panda_moveit_config's initial_positions.yaml) — without this,
+       joints default to a state that (for fer_joint4) sits essentially
+       exactly on its upper limit, causing MoveIt's CheckStartStateBounds
+       to reject the start state due to floating-point boundary issues. -->
   <ros2_control name="InspectraPandaSystem" type="system">
     <hardware>
       <plugin>gz_ros2_control/GazeboSimSystem</plugin>
     </hardware>
-    <xacro:macro name="fer_joint_interface" params="joint_name">
+    <xacro:macro name="fer_joint_interface" params="joint_name initial_value">
       <joint name="${joint_name}">
         <command_interface name="position"/>
-        <state_interface name="position"/>
+        <state_interface name="position">
+          <param name="initial_value">${initial_value}</param>
+        </state_interface>
         <state_interface name="velocity"/>
         <state_interface name="effort"/>
       </joint>
     </xacro:macro>
-    <xacro:fer_joint_interface joint_name="fer_joint1"/>
-    <xacro:fer_joint_interface joint_name="fer_joint2"/>
-    <xacro:fer_joint_interface joint_name="fer_joint3"/>
-    <xacro:fer_joint_interface joint_name="fer_joint4"/>
-    <xacro:fer_joint_interface joint_name="fer_joint5"/>
-    <xacro:fer_joint_interface joint_name="fer_joint6"/>
-    <xacro:fer_joint_interface joint_name="fer_joint7"/>
+    <xacro:fer_joint_interface joint_name="fer_joint1" initial_value="0.0"/>
+    <xacro:fer_joint_interface joint_name="fer_joint2" initial_value="-0.785"/>
+    <xacro:fer_joint_interface joint_name="fer_joint3" initial_value="0.0"/>
+    <xacro:fer_joint_interface joint_name="fer_joint4" initial_value="-2.356"/>
+    <xacro:fer_joint_interface joint_name="fer_joint5" initial_value="0.0"/>
+    <xacro:fer_joint_interface joint_name="fer_joint6" initial_value="1.571"/>
+    <xacro:fer_joint_interface joint_name="fer_joint7" initial_value="0.785"/>
   </ros2_control>
   <gazebo>

File: ros2_ws/src/inspectra_moveit_config/config/inspectra_panda.ros2_control.xacro (robot description, xacro)
@@ -8,50 +8,50 @@
                 <plugin>mock_components/GenericSystem</plugin>
             </hardware>
-            <joint name="fer_joint1">
+            <joint name="panda_joint1">
                 <command_interface name="position"/>
                 <state_interface name="position">
-                  <param name="initial_value">${initial_positions['fer_joint1']}</param>
+                  <param name="initial_value">${initial_positions['panda_joint1']}</param>
                 </state_interface>
                 <state_interface name="velocity"/>
             </joint>
-            <joint name="fer_joint2">
+            <joint name="panda_joint2">
                 <command_interface name="position"/>
                 <state_interface name="position">
-                  <param name="initial_value">${initial_positions['fer_joint2']}</param>
+                  <param name="initial_value">${initial_positions['panda_joint2']}</param>
                 </state_interface>
                 <state_interface name="velocity"/>
             </joint>
-            <joint name="fer_joint3">
+            <joint name="panda_joint3">
                 <command_interface name="position"/>
                 <state_interface name="position">
-                  <param name="initial_value">${initial_positions['fer_joint3']}</param>
+                  <param name="initial_value">${initial_positions['panda_joint3']}</param>
                 </state_interface>
                 <state_interface name="velocity"/>
             </joint>
-            <joint name="fer_joint4">
+            <joint name="panda_joint4">
                 <command_interface name="position"/>
                 <state_interface name="position">
-                  <param name="initial_value">${initial_positions['fer_joint4']}</param>
+                  <param name="initial_value">${initial_positions['panda_joint4']}</param>
                 </state_interface>
                 <state_interface name="velocity"/>
             </joint>
-            <joint name="fer_joint5">
+            <joint name="panda_joint5">
                 <command_interface name="position"/>
                 <state_interface name="position">
-                  <param name="initial_value">${initial_positions['fer_joint5']}</param>
+                  <param name="initial_value">${initial_positions['panda_joint5']}</param>
                 </state_interface>
                 <state_interface name="velocity"/>
             </joint>
-            <joint name="fer_joint6">
+            <joint name="panda_joint6">
                 <command_interface name="position"/>
                 <state_interface name="position">
-                  <param name="initial_value">${initial_positions['fer_joint6']}</param>
+                  <param name="initial_value">${initial_positions['panda_joint6']}</param>
                 </state_interface>
                 <state_interface name="velocity"/>
             </joint>
-            <joint name="fer_joint7">
+            <joint name="panda_joint7">
                 <command_interface name="position"/>
                 <state_interface name="position">
-                  <param name="initial_value">${initial_positions['fer_joint7']}</param>
+                  <param name="initial_value">${initial_positions['panda_joint7']}</param>
                 </state_interface>
                 <state_interface name="velocity"/>

Commit message: feat: GOOD/BAD PCB color-coded sorting (green/red), 4-leg brown table in RViz
- scene_manager.py: table+4 legs with brown coloring, set_object_color()
  via real PlanningScene publisher (uses motion_planner_node's own node)
- motion_planner.py: unified cycle handles both GOOD and BAD -- picks,
  colors the block green (GOOD) or red (BAD), sorts to matching bin.
  Fixes earlier bug where BAD boards dragged the object to HOME instead
  of completing a proper sort.
- Added inspectra_industrial_demo.launch.py (combined Gazebo+bringup+
  perception launch) and test files from a prior session -- kept as-is,
  not yet verified against known Gazebo+bringup controller-name conflict

File: ros2_ws/src/inspectra_description/urdf/inspectra_panda.urdf.xacro (robot description, xacro)
@@ -10,38 +10,17 @@
     robot_type="fer"
     connected_to="world"
-    hand="false"
-    gazebo="false"
+    hand="true"
+    ee_id="franka_hand"
+    gazebo="true"
     no_prefix="false"
     arm_prefix=""
   />
-  <!-- ros2_control interface: exposes each joint's position command/state
-       so gz_ros2_control's plugin (below) can drive them in simulation.
-       initial_value set explicitly per joint (matching moveit_resources_
-       panda_moveit_config's initial_positions.yaml) — without this,
-       joints default to a state that (for fer_joint4) sits essentially
-       exactly on its upper limit, causing MoveIt's CheckStartStateBounds
-       to reject the start state due to floating-point boundary issues. -->
-  <ros2_control name="InspectraPandaSystem" type="system">
-    <hardware>
-      <plugin>gz_ros2_control/GazeboSimSystem</plugin>
-    </hardware>
-    <xacro:macro name="fer_joint_interface" params="joint_name initial_value">
-      <joint name="${joint_name}">
-        <command_interface name="position"/>
-        <state_interface name="position">
-          <param name="initial_value">${initial_value}</param>
-        </state_interface>
-        <state_interface name="velocity"/>
-        <state_interface name="effort"/>
-      </joint>
-    </xacro:macro>
-    <xacro:fer_joint_interface joint_name="fer_joint1" initial_value="0.0"/>
-    <xacro:fer_joint_interface joint_name="fer_joint2" initial_value="-0.785"/>
-    <xacro:fer_joint_interface joint_name="fer_joint3" initial_value="0.0"/>
-    <xacro:fer_joint_interface joint_name="fer_joint4" initial_value="-2.356"/>
-    <xacro:fer_joint_interface joint_name="fer_joint5" initial_value="0.0"/>
-    <xacro:fer_joint_interface joint_name="fer_joint6" initial_value="1.571"/>
-    <xacro:fer_joint_interface joint_name="fer_joint7" initial_value="0.785"/>
-  </ros2_control>
+  <gazebo reference="panda_link0">
+    <static>true</static>
+    <kinematic>true</kinematic>
+  </gazebo>
+  <gazebo reference="fer_joint_world">
+    <preserveFixedJoint>true</preserveFixedJoint>
+  </gazebo>
   <gazebo>
     <plugin filename="gz_ros2_control-system" name="gz_ros2_control::GazeboSimROS2ControlPlugin">
